File: InterNoC.kicad_pcb (KiCad board)
At the start: 6 copper layers, 100 x 120 mm, 365 parts, among them J1 BARREL_JACK, J10 I2C_MASTER_3, J11 I2C_MASTER_4, J12 UART_MASTER_1, J13 SPI_MASTER_1, J14 SPI_MASTER_2, J15 SPI_MASTER_3, J16 I2C_SLAVE_1, J17 I2C_SLAVE_2, J18 I2C_SLAVE_3, J19 I2C_SLAVE_4, J2 CONN_01X02, J20 UART_SLAVE_1, J21 SPI_SLAVE_1, J22 SPI_SLAVE_2, J23 SPI_SLAVE_3, J24 I2C_SLAVE_5, J25 I2C_SLAVE_6, J26 I2C_SLAVE_7, J27 I2C_SLAVE_8, J28 UART_SLAVE_2, J29 SPI_SLAVE_4, J3 TEST_PW_IN, J30 SPI_SLAVE_5, J31 SPI_SLAVE_6, J32 JTAG HEADER, J4 TEST_GND, J5 TEST_1V8, J6 TEST_1V0, J7 TEST_3V3, J8 I2C_MASTER_1, J9 I2C_MASTER_2, Q1 FDV301N, Q2 Q_NMOS_DGS, SW1 SW_SPDT, SW2 RST_CONF, SW3 SW_Push, SW4 SW_Push, U1 TPS7A9101DSKT, U2 TPS7A9201DSKR, U3 xc7a35tfgg484, U4 ABRACON_ASDM1-100.000MHZ-LC-T, U5 S25FL128SAGBHIA00, U6 TPS7A9101DSKT

Commit message: pcb complete commit
the layout is complete. NOT checked & verified
Parts:
- removed C102, C103, C69, C70, C78, C79: 47nF X5R, Capacitors_SMD:C_0603_HandSoldering
- removed C58, C65, C66, C67, C68, C74, C75, C76, C77, C90, C93, C96, C99: 470nF X5R, Capacitors_SMD:C_0603_HandSoldering
- removed C59, C60, C63, C64, C72, C73, C84, C88: 4.7uF X5R, Capacitors_SMD:C_0805_HandSoldering
- removed C61, C62, C71, C82: 100uF X5R, Capacitors_SMD:C_1210_HandSoldering
- added C21: 100uF X5R, Capacitors_SMD:C_1210_HandSoldering, B.Cu at (107.7, 68.7)
- added C22: 100uF X5R, Capacitors_SMD:C_1210_HandSoldering, B.Cu at (110.8, 68.7)
- added C23: 100uF X5R, Capacitors_SMD:C_1210_HandSoldering, B.Cu at (97.5, 84.1)
- added C24: 100uF X5R, Capacitors_SMD:C_1210_HandSoldering, B.Cu at (122.2, 85.9)
- added C25: 4.7uF X5R, Capacitors_SMD:C_0805_HandSoldering, B.Cu at (103.2, 69.7)
- added C26: 4.7uF X5R, Capacitors_SMD:C_0805_HandSoldering, B.Cu at (113.2, 69.7)
- added C27: 4.7uF X5R, Capacitors_SMD:C_0805_HandSoldering, B.Cu at (98.5, 86.6)
- added C28: 4.7uF X5R, Capacitors_SMD:C_0805_HandSoldering, B.Cu at (121.3, 90.2)
- added C29: 4.7uF X5R, Capacitors_SMD:C_0805_HandSoldering, B.Cu at (105.1, 69.7)
- added C30: 4.7uF X5R, Capacitors_SMD:C_0805_HandSoldering, B.Cu at (115.0, 69.7)
- added C31: 4.7uF X5R, Capacitors_SMD:C_0805_HandSoldering, B.Cu at (98.5, 88.5)
- added REF**: MountingHole_3.2mm_M3, Mounting_Holes:MountingHole_3.2mm_M3, F.Cu at (62.2, 132.0)
- added REF**: VIA - 2mil, InterNoC:VIA_2mil, F.Cu at (139.1, 126.7)
- added REF**: VIA - 2mil, InterNoC:VIA_2mil, F.Cu at (112.4, 128.6)
- added REF**: VIA - 2mil, InterNoC:VIA_2mil, F.Cu at (111.8, 128.6)
- added REF**: VIA - 2mil, InterNoC:VIA_2mil, F.Cu at (112.4, 128.0)
- added REF**: VIA - 2mil, InterNoC:VIA_2mil, F.Cu at (111.8, 128.0)
- added REF**: VIA - 2mil, InterNoC:VIA_2mil, F.Cu at (112.4, 127.4)
- added REF**: VIA - 2mil, InterNoC:VIA_2mil, F.Cu at (111.8, 127.4)
- added REF**: VIA - 2mil, InterNoC:VIA_2mil, F.Cu at (112.4, 126.8)
- added REF**: VIA - 2mil, InterNoC:VIA_2mil, F.Cu at (69.7, 132.8)
- added REF**: VIA - 2mil, InterNoC:VIA_2mil, F.Cu at (69.1, 132.8)
- added REF**: MountingHole_3.2mm_M3, Mounting_Holes:MountingHole_3.2mm_M3, F.Cu at (70.2, 51.0)
- added REF**: VIA - 2mil, InterNoC:VIA_2mil, F.Cu at (68.5, 132.8)
- added REF**: VIA - 2mil, InterNoC:VIA_2mil, F.Cu at (69.7, 132.1)
- added REF**: VIA - 2mil, InterNoC:VIA_2mil, F.Cu at (69.1, 132.1)
- added REF**: VIA - 2mil, InterNoC:VIA_2mil, F.Cu at (68.5, 132.1)
- added REF**: VIA - 2mil, InterNoC:VIA_2mil, F.Cu at (69.7, 131.3)
- added REF**: VIA - 2mil, InterNoC:VIA_2mil, F.Cu at (69.1, 131.3)
- added REF**: VIA - 2mil, InterNoC:VIA_2mil, F.Cu at (68.5, 131.3)
- added REF**: VIA - 2mil, InterNoC:VIA_2mil, F.Cu at (69.7, 130.6)
- added REF**: VIA - 2mil, InterNoC:VIA_2mil, F.Cu at (69.1, 130.6)
- added REF**: VIA - 2mil, InterNoC:VIA_2mil, F.Cu at (68.5, 130.6)
- added REF**: MountingHole_3.2mm_M3, Mounting_Holes:MountingHole_3.2mm_M3, F.Cu at (150.2, 51.0)
- added REF**: VIA - 2mil, InterNoC:VIA_2mil, F.Cu at (69.7, 129.8)
- added REF**: VIA - 2mil, InterNoC:VIA_2mil, F.Cu at (69.1, 129.8)
- added REF**: VIA - 2mil, InterNoC:VIA_2mil, F.Cu at (68.5, 129.8)
- added REF**: MountingHole_3.2mm_M3, Mounting_Holes:MountingHole_3.2mm_M3, F.Cu at (157.8, 132.0)
- added REF**: VIA - 2mil, InterNoC:VIA_2mil, F.Cu at (111.8, 126.8)
- added REF**: VIA - 2mil, InterNoC:VIA_2mil, F.Cu at (139.7, 127.9)
- added REF**: VIA - 2mil, InterNoC:VIA_2mil, F.Cu at (139.1, 127.9)
- added REF**: VIA - 2mil, InterNoC:VIA_2mil, F.Cu at (139.7, 127.3)
- added REF**: VIA - 2mil, InterNoC:VIA_2mil, F.Cu at (139.1, 127.3)
- added REF**: VIA - 2mil, InterNoC:VIA_2mil, F.Cu at (139.7, 126.7)
- C100, C101, C104, C105, C106, C107, C108, C109, C110, C111, C112, C113, C114, C35, C36, C37, C38, C39, C45, C47, C48, C49, C51, C52, C53, C54, C80, C81, C83, C85, C86, C87, C89, C91, C92, C94, C95, C97, C98, L4, L5: moved to B.Cu
- C32: value 100uF X5R -> 4.7uF X5R; footprint Capacitors_SMD:C_1210_HandSoldering -> Capacitors_SMD:C_0805_HandSoldering; moved to B.Cu
- C33, C34, C43, C44: value 4.7uF X5R -> 470nF X5R; footprint Capacitors_SMD:C_1210_HandSoldering -> Capacitors_SMD:C_0603_HandSoldering; moved to B.Cu
- C40, C41: value 47nF X5R -> 470nF X5R; moved to B.Cu
- C42: value 100uF X5R -> 470nF X5R; footprint Capacitors_SMD:C_1210_HandSoldering -> Capacitors_SMD:C_0603_HandSoldering; moved to B.Cu
- C50, C55, C56, C57: value 470nF X5R -> 47nF X5R; moved to B.Cu
- J3, J4, J5, J6, J7: footprint Wire_Pads:SolderWirePad_single_1mmDrill -> InterNoC:test_point_single
- U3: value xc7a35tfgg484 -> xc7a35tftg256; footprint InterNoC:XC7A35T-1FGG484C -> InterNoC:XC7A35T-1FTG256C
- moved R114 476.7 mm to (63.4, 138.0)
- moved D94 467.1 mm to (67.8, 140.2), turned to 180 degrees
- moved R116 463.1 mm to (71.4, 138.0)
- moved R117 456.0 mm to (75.4, 138.0)
- moved R115 452.2 mm to (67.4, 138.0)
- moved D96 449.4 mm to (77.4, 140.2), turned to 180 degrees
- moved D93 449.2 mm to (63.0, 140.2), turned to 180 degrees
- moved D95 447.8 mm to (72.6, 140.2), turned to 180 degrees
- moved D92 443.0 mm to (82.8, 143.2), turned to 180 degrees
- moved R111 442.5 mm to (82.4, 141.4), turned to 180 degrees
- moved C107 429.8 mm to (104.5, 91.6), turned to 180 degrees
- moved C114 428.0 mm to (99.2, 77.8), turned to 180 degrees
- moved C105 424.9 mm to (101.8, 96.8), turned to 270 degrees
- moved C108 424.2 mm to (109.2, 95.0), turned to 270 degrees
- moved C81 422.3 mm to (96.8, 93.8), turned to 180 degrees
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Connections:
- net Net-(D33-Pad1) renamed SPI_MASTER_2_MISO
- C100 pad 1: /Artix7/VCC1V0 -> /Artix7/VCC1V8
- C104 pad 1: /Artix7/VCC1V0 -> /Artix7/VCC1V8
- C106 pad 1: /Artix7/VCC1V0 -> /Artix7/VCC1V8
- C111 pad 1: /Artix7/VCC1V0 -> /Artix7/VCC1V8
- C12 pad 1: Net-(C12-Pad1) -> /Artix7/VCC1V8
- C5 pad 1: Net-(C12-Pad1) -> /Artix7/VCC1V8
- C8 pad 1: Net-(C12-Pad1) -> /Artix7/VCC1V8
- C86 pad 1: /Artix7/VCC1V0 -> /Artix7/VCC1V8
- C91 pad 1: /Artix7/VCC1V0 -> /Artix7/VCC1V8
- C94 pad 1: /Artix7/VCC1V0 -> /Artix7/VCC1V8
- C97 pad 1: /Artix7/VCC1V0 -> /Artix7/VCC1V8
- D26 pad 1: /MasterInterfaces/SPI_MASTER_1_SCLK -> SPI_MASTER_1_SCLK
- D27 pad 1: /MasterInterfaces/SPI_MASTER_2_SCLK -> SPI_MASTER_2_SCLK
- D28 pad 1: /MasterInterfaces/SPI_MASTER_3_SCLK -> SPI_MASTER_3_SCLK
- D29 pad 1: Net-(D29-Pad1) -> SPI_MASTER_1_MOSI
- D30 pad 1: Net-(D30-Pad1) -> SPI_MASTER_2_MOSI
- D31 pad 1: Net-(D31-Pad1) -> SPI_MASTER_3_MOSI
- D32 pad 1: Net-(D32-Pad1) -> SPI_MASTER_1_MISO
- D34 pad 1: Net-(D34-Pad1) -> SPI_MASTER_3_MISO
- D35 pad 1: Net-(D35-Pad1) -> I2C_MASTER_1_SDA
- D36 pad 1: Net-(D36-Pad1) -> SPI_MASTER_1_CS
- D37 pad 1: Net-(D37-Pad1) -> SPI_MASTER_2_CS
- D38 pad 1: Net-(D38-Pad1) -> SPI_MASTER_3_CS
- D39 pad 1: Net-(D39-Pad1) -> I2C_MASTER_1_SCL
- D40 pad 1: Net-(D40-Pad1) -> I2C_MASTER_2_SDA
- D41 pad 1: Net-(D41-Pad1) -> I2C_MASTER_2_SCL
- D42 pad 1: Net-(D42-Pad1) -> I2C_MASTER_3_SDA
- D43 pad 1: Net-(D43-Pad1) -> I2C_MASTER_3_SCL
- D44 pad 1: Net-(D44-Pad1) -> I2C_MASTER_4_SDA
- D45 pad 1: Net-(D45-Pad1) -> I2C_MASTER_4_SCL
- D46 pad 1: Net-(D46-Pad1) -> UART_MASTER_1_TX
- D47 pad 1: Net-(D47-Pad1) -> UART_MASTER_1_RX
- D48 pad 1: Net-(D48-Pad1) -> I2C_SLAVE_1_SDA
- D49 pad 1: Net-(D49-Pad1) -> I2C_SLAVE_1_SCL
- D50 pad 1: Net-(D50-Pad1) -> SPI_SLAVE_1_SCLK
- D51 pad 1: Net-(D51-Pad1) -> I2C_SLAVE_2_SDA
- D52 pad 1: Net-(D52-Pad1) -> SPI_SLAVE_1_MOSI
- D53 pad 1: Net-(D53-Pad1) -> I2C_SLAVE_2_SCL
- D54 pad 1: Net-(D54-Pad1) -> SPI_SLAVE_1_MISO
- D55 pad 1: Net-(D55-Pad1) -> I2C_SLAVE_3_SDA
- D56 pad 1: Net-(D56-Pad1) -> SPI_SLAVE_1_CS
- D57 pad 1: Net-(D57-Pad1) -> I2C_SLAVE_3_SCL
- D58 pad 1: Net-(D58-Pad1) -> SPI_SLAVE_2_SCLK
- D59 pad 1: Net-(D59-Pad1) -> I2C_SLAVE_4_SDA
- D60 pad 1: Net-(D60-Pad1) -> SPI_SLAVE_2_MOSI
- D61 pad 1: Net-(D61-Pad1) -> I2C_SLAVE_4_SCL
- D62 pad 1: Net-(D62-Pad1) -> SPI_SLAVE_2_MISO
- D63 pad 1: Net-(D63-Pad1) -> UART_SLAVE_1_TX
- D64 pad 1: Net-(D64-Pad1) -> SPI_SLAVE_2_CS
- D65 pad 1: Net-(D65-Pad1) -> UART_SLAVE_1_RX
- D66 pad 1: Net-(D66-Pad1) -> SPI_SLAVE_3_SCLK
- D67 pad 1: Net-(D67-Pad1) -> SPI_SLAVE_3_MOSI
- D68 pad 1: Net-(D68-Pad1) -> SPI_SLAVE_3_MISO
- D69 pad 1: Net-(D69-Pad1) -> SPI_SLAVE_3_CS
- D70 pad 1: Net-(D70-Pad1) -> I2C_SLAVE_5_SDA
- D71 pad 1: Net-(D71-Pad1) -> SPI_SLAVE_4_SCLK
- D72 pad 1: Net-(D72-Pad1) -> I2C_SLAVE_5_SCL
- D73 pad 1: Net-(D73-Pad1) -> SPI_SLAVE_4_MOSI
- D74 pad 1: Net-(D74-Pad1) -> I2C_SLAVE_6_SDA
- D75 pad 1: Net-(D75-Pad1) -> SPI_SLAVE_4_MISO
- D76 pad 1: Net-(D76-Pad1) -> I2C_SLAVE_6_SCL
- D77 pad 1: Net-(D77-Pad1) -> SPI_SLAVE_4_CS
- D78 pad 1: Net-(D78-Pad1) -> I2C_SLAVE_7_SDA
- D79 pad 1: Net-(D79-Pad1) -> SPI_SLAVE_5_SCLK
- D80 pad 1: Net-(D80-Pad1) -> I2C_SLAVE_7_SCL
- D81 pad 1: Net-(D81-Pad1) -> SPI_SLAVE_5_MOSI
- D82 pad 1: Net-(D82-Pad1) -> I2C_SLAVE_8_SDA
- D83 pad 1: Net-(D83-Pad1) -> SPI_SLAVE_5_MISO
- D84 pad 1: Net-(D84-Pad1) -> I2C_SLAVE_8_SCL
- D85 pad 1: Net-(D85-Pad1) -> SPI_SLAVE_5_CS
- D86 pad 1: Net-(D86-Pad1) -> UART_SLAVE_2_TX
- D87 pad 1: Net-(D87-Pad1) -> SPI_SLAVE_6_SCLK
- D88 pad 1: Net-(D88-Pad1) -> UART_SLAVE_2_RX
- D89 pad 1: Net-(D89-Pad1) -> SPI_SLAVE_6_MOSI
- D90 pad 1: Net-(D90-Pad1) -> SPI_SLAVE_6_MISO
- D91 pad 1: Net-(D91-Pad1) -> SPI_SLAVE_6_CS
- J5 pad 1: Net-(C12-Pad1) -> /Artix7/VCC1V8
- L4 pad 2: /Artix7/VCC1V0 -> /Artix7/VCC1V8
- R100 pad 1: Net-(D75-Pad1) -> SPI_SLAVE_4_MISO
- R101 pad 1: Net-(D77-Pad1) -> SPI_SLAVE_4_CS
- R102 pad 1: Net-(D79-Pad1) -> SPI_SLAVE_5_SCLK
- R103 pad 1: Net-(D81-Pad1) -> SPI_SLAVE_5_MOSI
- R104 pad 1: Net-(D83-Pad1) -> SPI_SLAVE_5_MISO
- R105 pad 1: Net-(D85-Pad1) -> SPI_SLAVE_5_CS
- R106 pad 1: Net-(D87-Pad1) -> SPI_SLAVE_6_SCLK
- R107 pad 1: Net-(D89-Pad1) -> SPI_SLAVE_6_MOSI
- R108 pad 1: Net-(D90-Pad1) -> SPI_SLAVE_6_MISO
- R109 pad 1: Net-(D91-Pad1) -> SPI_SLAVE_6_CS
- R118 pad 1: Net-(R118-Pad1) -> GP_BTN_1
- R119 pad 1: Net-(R119-Pad1) -> GP_BTN_2
- R20 pad 1: Net-(R20-Pad1) -> LED_1
- R21 pad 1: Net-(R21-Pad1) -> LED_2
- R22 pad 1: Net-(R22-Pad1) -> LED_3
- R23 pad 1: Net-(R23-Pad1) -> LED_4
- R24 pad 1: Net-(R24-Pad1) -> LED_5
- R25 pad 1: Net-(R25-Pad1) -> LED_6
- R26 pad 1: Net-(R26-Pad1) -> LED_7
- R27 pad 1: Net-(R27-Pad1) -> LED_8
- R28 pad 1: Net-(R28-Pad1) -> LED_9
- R29 pad 1: Net-(R29-Pad1) -> LED_10
- R30 pad 1: Net-(R30-Pad1) -> LED_11
- R31 pad 1: Net-(R31-Pad1) -> LED_12
- R32 pad 1: Net-(R32-Pad1) -> LED_13
- R33 pad 1: Net-(R33-Pad1) -> LED_14
- R34 pad 1: Net-(R34-Pad1) -> LED_15
- R35 pad 1: Net-(R35-Pad1) -> LED_16
- R36 pad 1: Net-(R36-Pad1) -> LED_17
- R37 pad 1: Net-(R37-Pad1) -> LED_18
- R38 pad 1: Net-(R38-Pad1) -> LED_19
- R39 pad 1: Net-(R39-Pad1) -> LED_20
- R40 pad 1: Net-(R40-Pad1) -> LED_21
- R41 pad 1: Net-(R41-Pad1) -> LED_22
- R42 pad 1: Net-(R42-Pad1) -> LED_23
- R43 pad 1: Net-(R43-Pad1) -> LED_24
- R44 pad 2: Net-(D35-Pad1) -> I2C_MASTER_1_SDA
- R45 pad 2: Net-(D39-Pad1) -> I2C_MASTER_1_SCL
- R46 pad 2: Net-(D40-Pad1) -> I2C_MASTER_2_SDA
- R47 pad 2: Net-(D41-Pad1) -> I2C_MASTER_2_SCL
- R48 pad 2: Net-(D42-Pad1) -> I2C_MASTER_3_SDA
- R49 pad 2: Net-(D43-Pad1) -> I2C_MASTER_3_SCL
- R5 pad 1: Net-(C12-Pad1) -> /Artix7/VCC1V8
- R50 pad 2: Net-(D44-Pad1) -> I2C_MASTER_4_SDA
- R51 pad 2: Net-(D45-Pad1) -> I2C_MASTER_4_SCL
- R52 pad 2: Net-(D46-Pad1) -> UART_MASTER_1_TX
- R53 pad 2: Net-(D47-Pad1) -> UART_MASTER_1_RX
- R54 pad 2: /MasterInterfaces/SPI_MASTER_1_SCLK -> SPI_MASTER_1_SCLK
- R55 pad 2: Net-(D29-Pad1) -> SPI_MASTER_1_MOSI
- R56 pad 2: Net-(D32-Pad1) -> SPI_MASTER_1_MISO
- R57 pad 2: Net-(D36-Pad1) -> SPI_MASTER_1_CS
- R58 pad 2: /MasterInterfaces/SPI_MASTER_2_SCLK -> SPI_MASTER_2_SCLK
- R59 pad 2: Net-(D30-Pad1) -> SPI_MASTER_2_MOSI
- R61 pad 2: Net-(D37-Pad1) -> SPI_MASTER_2_CS
- R62 pad 2: /MasterInterfaces/SPI_MASTER_3_SCLK -> SPI_MASTER_3_SCLK
- R63 pad 2: Net-(D31-Pad1) -> SPI_MASTER_3_MOSI
- R64 pad 2: Net-(D34-Pad1) -> SPI_MASTER_3_MISO
- R65 pad 2: Net-(D38-Pad1) -> SPI_MASTER_3_CS
- R66 pad 1: Net-(D57-Pad1) -> I2C_SLAVE_3_SCL
- R67 pad 1: Net-(D48-Pad1) -> I2C_SLAVE_1_SDA
- R68 pad 1: Net-(D49-Pad1) -> I2C_SLAVE_1_SCL
- R69 pad 1: Net-(D51-Pad1) -> I2C_SLAVE_2_SDA
- R70 pad 1: Net-(D53-Pad1) -> I2C_SLAVE_2_SCL
- R71 pad 1: Net-(D55-Pad1) -> I2C_SLAVE_3_SDA
- R72 pad 1: Net-(D59-Pad1) -> I2C_SLAVE_4_SDA
- R73 pad 1: Net-(D61-Pad1) -> I2C_SLAVE_4_SCL
- R74 pad 1: Net-(D63-Pad1) -> UART_SLAVE_1_TX
- R75 pad 1: Net-(D65-Pad1) -> UART_SLAVE_1_RX
- R76 pad 1: Net-(D50-Pad1) -> SPI_SLAVE_1_SCLK
- R77 pad 1: Net-(D52-Pad1) -> SPI_SLAVE_1_MOSI
- R78 pad 1: Net-(D54-Pad1) -> SPI_SLAVE_1_MISO
- R79 pad 1: Net-(D56-Pad1) -> SPI_SLAVE_1_CS
- R80 pad 1: Net-(D58-Pad1) -> SPI_SLAVE_2_SCLK
- R81 pad 1: Net-(D60-Pad1) -> SPI_SLAVE_2_MOSI
- R82 pad 1: Net-(D62-Pad1) -> SPI_SLAVE_2_MISO
- R83 pad 1: Net-(D64-Pad1) -> SPI_SLAVE_2_CS
- R84 pad 1: Net-(D66-Pad1) -> SPI_SLAVE_3_SCLK
- R85 pad 1: Net-(D67-Pad1) -> SPI_SLAVE_3_MOSI
- R86 pad 1: Net-(D68-Pad1) -> SPI_SLAVE_3_MISO
- R87 pad 1: Net-(D69-Pad1) -> SPI_SLAVE_3_CS
- R88 pad 1: Net-(D70-Pad1) -> I2C_SLAVE_5_SDA
- R89 pad 1: Net-(D72-Pad1) -> I2C_SLAVE_5_SCL
- R90 pad 1: Net-(D74-Pad1) -> I2C_SLAVE_6_SDA
- R91 pad 1: Net-(D76-Pad1) -> I2C_SLAVE_6_SCL
- R92 pad 1: Net-(D78-Pad1) -> I2C_SLAVE_7_SDA
- R93 pad 1: Net-(D80-Pad1) -> I2C_SLAVE_7_SCL
- R94 pad 1: Net-(D82-Pad1) -> I2C_SLAVE_8_SDA
- R95 pad 1: Net-(D84-Pad1) -> I2C_SLAVE_8_SCL
- R96 pad 1: Net-(D86-Pad1) -> UART_SLAVE_2_TX
- R97 pad 1: Net-(D88-Pad1) -> UART_SLAVE_2_RX
- R98 pad 1: Net-(D71-Pad1) -> SPI_SLAVE_4_SCLK
- R99 pad 1: Net-(D73-Pad1) -> SPI_SLAVE_4_MOSI
- U1 pad 1: Net-(C12-Pad1) -> /Artix7/VCC1V8
- U1 pad 2: Net-(C12-Pad1) -> /Artix7/VCC1V8
- U3 pad A1: Net-(D32-Pad1) -> GND
- U3 pad A10: GND -> LED_14
- U3 pad A12: GND -> LED_17
- U3 pad A13: Net-(U3-PadA13) -> LED_19
- U3 pad A14: Net-(U3-PadA14) -> LED_20
- U3 pad A15: Net-(U3-PadA15) -> LED_22
- U3 pad A16: Net-(U3-PadA16) -> /Artix7/VCC3V3
- U3 pad A2: GND -> LED_3
- U3 pad A3: GND -> LED_4
- U3 pad A4: GND -> LED_6
- U3 pad A5: GND -> LED_8
- U3 pad A6: GND -> /Artix7/VCC3V3
- U3 pad A7: GND -> LED_11
- U3 pad A8: GND -> LED_12
- U3 pad A9: GND -> Net-(U3-PadA9)
- U3 pad B1: Net-(D36-Pad1) -> LED_1
- U3 pad B10: GND -> LED_15
- U3 pad B11: GND -> LED_16
- U3 pad B12: GND -> LED_18
- U3 pad B13: Net-(U3-PadB13) -> /Artix7/VCC3V3
- U3 pad B14: /Artix7/VCC3V3 -> LED_21
- U3 pad B15: Net-(U3-PadB15) -> LED_23
- U3 pad B16: Net-(U3-PadB16) -> LED_24
- U3 pad B2: Net-(U3-PadB2) -> LED_2
- U3 pad B3: GND -> /Artix7/VCC3V3
- U3 pad B4: GND -> LED_5
- U3 pad B5: GND -> LED_7
- U3 pad B6: GND -> LED_9
- U3 pad B7: GND -> LED_10
- U3 pad B9: GND -> LED_13
- U3 pad C1: /Artix7/VCC3V3 -> SPI_MASTER_1_CS
- U3 pad C10: GND -> /Artix7/VCC3V3
- U3 pad C11: GND -> Net-(U3-PadC11)
- U3 pad C12: GND -> Net-(U3-PadC12)
- U3 pad C13: Net-(U3-PadC13) -> CLOCK
- U3 pad C14: Net-(U3-PadC14) -> SPI_SLAVE_1_MOSI
- U3 pad C15: Net-(U3-PadC15) -> GND
- U3 pad C16: GND -> SPI_SLAVE_1_SCLK
- U3 pad C2: Net-(D30-Pad1) -> SPI_MASTER_1_MISO
- U3 pad C3: GND -> SPI_MASTER_1_SCLK
- U3 pad C4: GND -> SPI_MASTER_1_MOSI
- U3 pad C6: GND -> Net-(U3-PadC6)
- U3 pad C7: GND -> Net-(U3-PadC7)
- U3 pad C8: GND -> Net-(U3-PadC8)
- U3 pad C9: GND -> Net-(U3-PadC9)
- U3 pad D10: GND -> Net-(U3-PadD10)
- U3 pad D11: GND -> Net-(U3-PadD11)
- U3 pad D13: GND -> Net-(U3-PadD13)
- U3 pad D15: Net-(U3-PadD15) -> SPI_SLAVE_1_CS
- U3 pad D16: Net-(U3-PadD16) -> SPI_SLAVE_1_MISO
- U3 pad D2: Net-(U3-PadD2) -> GND
- U3 pad D3: GND -> SPI_MASTER_2_MOSI
- U3 pad D4: GND -> SPI_MASTER_2_SCLK
- U3 pad D5: GND -> SPI_MASTER_2_CS
- U3 pad D6: GND -> Net-(U3-PadD6)
- U3 pad D7: GND -> /Artix7/VCC3V3
- U3 pad D8: GND -> Net-(U3-PadD8)
- U3 pad D9: GND -> Net-(U3-PadD9)
- U3 pad E1: Net-(D37-Pad1) -> SPI_MASTER_3_MOSI
- U3 pad E10: GND -> /Artix7/VCC1V0
- U3 pad E11: GND -> Net-(U3-PadE11)
- U3 pad E12: /Artix7/VCC1V0 -> Net-(U3-PadE12)
- U3 pad E14: Net-(U3-PadE14) -> /Artix7/VCC3V3
- U3 pad E15: /Artix7/VCC3V3 -> SPI_SLAVE_2_SCLK
- U3 pad E16: Net-(U3-PadE16) -> SPI_SLAVE_2_MOSI
- U3 pad E2: Net-(D31-Pad1) -> SPI_MASTER_3_SCLK
- U3 pad E3: Net-(U3-PadE3) -> SPI_MASTER_3_MISO
- U3 pad E4: GND -> /Artix7/VCC3V3
- U3 pad E5: GND -> SPI_MASTER_3_CS
- U3 pad E6: GND -> Net-(U3-PadE6)
- U3 pad E7: GND -> /Artix7/VCC3V3
- U3 pad E8: GND -> Net-(U3-PadE8)
- U3 pad F1: Net-(D34-Pad1) -> /Artix7/VCC3V3
- U3 pad F11: GND -> /Artix7/VCC1V0
- U3 pad F12: /Artix7/VCC3V3 -> Net-(U3-PadF12)
- U3 pad F14: Net-(U3-PadF14) -> SPI_SLAVE_2_CS
- U3 pad F15: Net-(U3-PadF15) -> SPI_SLAVE_2_MISO
- U3 pad F16: Net-(U3-PadF16) -> GND
- U3 pad F2: /Artix7/VCC3V3 -> I2C_MASTER_1_SDA
- U3 pad F3: Net-(U3-PadF3) -> I2C_MASTER_1_SCL
- U3 pad F5: GND -> Net-(U3-PadF5)
- U3 pad F7: GND -> /Artix7/VCC1V0
- U3 pad F8: GND -> /Artix7/VCC1V8
- U3 pad F9: GND -> /Artix7/VCC1V0
- U3 pad G1: Net-(D38-Pad1) -> I2C_MASTER_2_SDA
- U3 pad G10: GND -> /Artix7/VCC1V8
- U3 pad G11: Net-(Q2-Pad2) -> Net-(U3-PadG11)
- U3 pad G12: GND -> Net-(U3-PadG12)
- U3 pad G13: Net-(R22-Pad1) -> GND
- U3 pad G14: GND -> Net-(U3-PadG14)
- U3 pad G15: Net-(R25-Pad1) -> SPI_SLAVE_3_MOSI
- U3 pad G16: Net-(R24-Pad1) -> SPI_SLAVE_3_SCLK
- U3 pad G2: Net-(U3-PadG2) -> I2C_MASTER_2_SCL
- U3 pad G3: /MasterInterfaces/SPI_MASTER_1_SCLK -> GND
- U3 pad G5: GND -> Net-(U3-PadG5)
- U3 pad G6: GND -> /Artix7/VCC1V0
- U3 pad G7: GND -> /Artix7/GNDADC
- U3 pad G8: GND -> /Artix7/VCCADC
- U3 pad H1: GND -> I2C_MASTER_3_SDA
- U3 pad H10: /Artix7/VCC1V0 -> Net-(Q2-Pad2)
- U3 pad H11: GND -> Net-(U3-PadH11)
- U3 pad H12: /Artix7/VCC1V0 -> Net-(U3-PadH12)
- U3 pad H13: Net-(R23-Pad1) -> Net-(U3-PadH13)
- U3 pad H14: Net-(R26-Pad1) -> SPI_SLAVE_3_MISO
- U3 pad H15: Net-(R30-Pad1) -> /Artix7/VCC3V3
- U3 pad H16: /Artix7/VCC3V3 -> SPI_SLAVE_3_CS
- U3 pad H2: Net-(U3-PadH2) -> I2C_MASTER_3_SCL
- U3 pad H3: /MasterInterfaces/SPI_MASTER_2_SCLK -> Net-(U3-PadH3)
- U3 pad H6: /Artix7/VCC3V3 -> GND
- U3 pad H7: GND -> /Artix7/GNDADC
- U3 pad H8: /Artix7/VCC1V0 -> /Artix7/GNDADC
- U3 pad H9: GND -> /Artix7/VCC1V0
- U3 pad J1: Net-(U3-PadJ1) -> I2C_MASTER_4_SDA
- U3 pad J10: GND -> /Artix7/VCC1V8
- U3 pad J11: /Artix7/VCC1V0 -> GND
- U3 pad J12: GND -> /Artix7/VCC3V3
- U3 pad J13: /Artix7/VCC3V3 -> Net-(U3-PadJ13)
- U3 pad J14: Net-(R27-Pad1) -> Net-(U3-PadJ14)
- U3 pad J15: Net-(R31-Pad1) -> I2C_SLAVE_1_SCL
- U3 pad J16: Net-(R20-Pad1) -> I2C_SLAVE_1_SDA
- U3 pad J2: Net-(U3-PadJ2) -> /Artix7/VCC3V3
- U3 pad J3: /Artix7/VCC3V3 -> I2C_MASTER_4_SCL
- U3 pad J6: Net-(D42-Pad1) -> /Artix7/VCC1V0
- U3 pad J7: /Artix7/VCC1V0 -> /Artix7/GNDADC
- U3 pad J8: GND -> /Artix7/GNDADC
- U3 pad J9: /Artix7/VCC1V0 -> GND
- U3 pad K1: Net-(U3-PadK1) -> UART_MASTER_1_TX
- U3 pad K10: /Artix7/VCCADC -> Net-(R113-Pad2)
- U3 pad K11: GND -> /Artix7/VCC1V8
- U3 pad K12: /Artix7/VCC1V0 -> Net-(U3-PadK12)
- U3 pad K14: Net-(U3-PadK14) -> GND
- U3 pad K15: GND -> I2C_SLAVE_2_SCL
- U3 pad K16: Net-(U3-PadK16) -> I2C_SLAVE_2_SDA
- U3 pad K2: Net-(U3-PadK2) -> UART_MASTER_1_RX
- U3 pad K3: /MasterInterfaces/SPI_MASTER_3_SCLK -> Net-(U3-PadK3)
- U3 pad K4: Net-(U3-PadK4) -> GND
- U3 pad K5: GND -> Net-(U3-PadK5)
- U3 pad K6: Net-(D43-Pad1) -> GND
- U3 pad K8: /Artix7/VCC1V0 -> GND
- U3 pad K9: /Artix7/GNDADC -> /Artix7/VCC1V0
- U3 pad L1: Net-(D35-Pad1) -> GND
- U3 pad L10: /Artix7/GNDADC -> /Artix7/VCC1V8
- U3 pad L11: /Artix7/VCC1V0 -> GND
- U3 pad L12: Net-(U3-PadL12) -> Net-(R110-Pad2)
- U3 pad L15: Net-(U3-PadL15) -> GND
- U3 pad L16: Net-(U3-PadL16) -> /Artix7/VCC3V3
- U3 pad L2: GND -> Net-(U3-PadL2)
- U3 pad L4: Net-(D44-Pad1) -> Net-(U3-PadL4)
- U3 pad L5: Net-(D45-Pad1) -> Net-(U3-PadL5)
- U3 pad L6: Net-(D29-Pad1) -> /Artix7/VCC3V3
- U3 pad L7: /Artix7/VCC1V0 -> /Artix7/TCK
- U3 pad L8: GND -> /Artix7/VCC1V0
- U3 pad L9: /Artix7/GNDADC -> Net-(R112-Pad2)
- U3 pad M1: Net-(D39-Pad1) -> GP_BTN_1
- U3 pad M10: /Artix7/GNDADC -> GND
- U3 pad M12: /Artix7/VCC1V0 -> Net-(U3-PadM12)
- U3 pad M13: Net-(U3-PadM13) -> /Artix7/VCC3V3
- U3 pad M14: /Artix7/VCC3V3 -> Net-(U3-PadM14)
- U3 pad M15: Net-(U3-PadM15) -> I2C_SLAVE_3_SCL
- U3 pad M16: Net-(U3-PadM16) -> I2C_SLAVE_3_SDA
- U3 pad M2: Net-(D40-Pad1) -> Net-(U3-PadM2)
- U3 pad M3: Net-(D41-Pad1) -> /Artix7/VCC3V3
- U3 pad M4: /Artix7/VCC3V3 -> Net-(U3-PadM4)
- U3 pad M7: GND -> /Artix7/TMS
- U3 pad M8: /Artix7/VCC1V0 -> GND
- U3 pad M9: /Artix7/GNDADC -> /Artix7/VCC3V3
- U3 pad N1: /Artix7/VCC3V3 -> GP_BTN_2
- U3 pad N10: GND -> /Artix7/VCC3V3
- U3 pad N11: /Artix7/VCC1V0 -> Net-(U3-PadN11)
- U3 pad N12: Net-(R112-Pad2) -> Net-(U3-PadN12)
- U3 pad N14: Net-(U3-PadN14) -> I2C_SLAVE_4_SCL
- U3 pad N15: Net-(D54-Pad1) -> GND
- U3 pad N16: GND -> I2C_SLAVE_4_SDA
- U3 pad N3: Net-(D46-Pad1) -> Net-(U3-PadN3)
- U3 pad N4: Net-(D47-Pad1) -> Net-(U3-PadN4)
- U3 pad N5: Net-(U3-PadN5) -> GND
- U3 pad N6: GND -> Net-(U3-PadN6)
- U3 pad N7: /Artix7/VCC1V0 -> /Artix7/TDI
- U3 pad N8: GND -> /Artix7/TDO
- U3 pad N9: GND -> Net-(U3-PadN9)
- U3 pad P1: Net-(U3-PadP1) -> SPI_SLAVE_4_SCLK
- U3 pad P10: /Artix7/VCC1V0 -> Net-(U3-PadP10)
- U3 pad P11: GND -> UART_SLAVE_2_RX
- U3 pad P12: /Artix7/VCC1V0 -> GND
- U3 pad P13: GND -> Net-(U3-PadP13)
- U3 pad P15: Net-(U3-PadP15) -> UART_SLAVE_1_RX
- U3 pad P16: Net-(U3-PadP16) -> UART_SLAVE_1_TX
- U3 pad P2: Net-(U3-PadP2) -> GND
- U3 pad P3: GND -> Net-(U3-PadP3)
- U3 pad P4: Net-(U3-PadP4) -> SPI_SLAVE_5_MISO
- U3 pad P6: Net-(U3-PadP6) -> SPI_SLAVE_6_CS
- U3 pad P7: GND -> /Artix7/VCC3V3
- U3 pad P8: /Artix7/VCC1V0 -> Net-(U3-PadP8)
- U3 pad P9: GND -> I2C_SLAVE_7_SCL
- U3 pad R1: Net-(U3-PadR1) -> SPI_SLAVE_4_MOSI
- U3 pad R10: GND -> I2C_SLAVE_8_SCL
- U3 pad R11: /Artix7/VCC1V0 -> UART_SLAVE_2_TX
- U3 pad R12: GND -> Net-(U3-PadR12)
- U3 pad R13: /Artix7/TDI -> Net-(U3-PadR13)
- U3 pad R14: Net-(U3-PadR14) -> /Artix7/VCC3V3
- U3 pad R15: /Artix7/VCC3V3 -> Net-(U3-PadR15)
- U3 pad R2: Net-(D85-Pad1) -> SPI_SLAVE_4_MISO
- U3 pad R3: Net-(U3-PadR3) -> SPI_SLAVE_5_SCLK
- U3 pad R4: Net-(D76-Pad1) -> /Artix7/VCC3V3
- U3 pad R5: /Artix7/VCC3V3 -> SPI_SLAVE_6_SCLK
- U3 pad R6: Net-(U3-PadR6) -> SPI_SLAVE_6_MISO
- U3 pad R7: /Artix7/VCC1V0 -> I2C_SLAVE_5_SCL
- U3 pad R8: GND -> I2C_SLAVE_6_SCL
- U3 pad R9: /Artix7/VCC1V0 -> GND
- U3 pad T1: Net-(U3-PadT1) -> /Artix7/VCC3V3
- U3 pad T10: /Artix7/VCC1V0 -> I2C_SLAVE_8_SDA
- U3 pad T11: GND -> /Artix7/VCC3V3
- U3 pad T12: /Artix7/VCC3V3 -> Net-(U3-PadT12)
- U3 pad T13: /Artix7/TMS -> Net-(U3-PadT13)
- U3 pad T14: Net-(U3-PadAA10) -> Net-(U3-PadT14)
- U3 pad T15: Net-(U3-PadAA10) -> Net-(U3-PadT15)
- U3 pad T16: Net-(U3-PadAA10) -> GND
- U3 pad T2: /Artix7/VCC3V3 -> SPI_SLAVE_4_CS
- U3 pad T3: Net-(D73-Pad1) -> SPI_SLAVE_5_MOSI
- U3 pad T4: Net-(D74-Pad1) -> SPI_SLAVE_5_CS
- U3 pad T5: Net-(D78-Pad1) -> SPI_SLAVE_6_MOSI
- U3 pad T6: Net-(D88-Pad1) -> GND
- U3 pad T7: GND -> I2C_SLAVE_5_SDA
- U3 pad T8: /Artix7/VCC1V0 -> I2C_SLAVE_6_SDA
- U3 pad T9: GND -> I2C_SLAVE_7_SDA
- U4 pad 3: Net-(U3-PadC17) -> CLOCK
- U5 pad B2: Net-(U3-PadL12) -> Net-(U3-PadE8)
- U5 pad D2: Net-(U3-PadR22) -> Net-(U3-PadJ14)
- U5 pad D3: Net-(U3-PadP22) -> Net-(U3-PadJ13)
Routing:
- net GND: track 0.00 -> 320.5 mm, vias 0 -> 234
- net Net-(Q2-Pad2): track 0.00 -> 107.4 mm, vias 0 -> 3
- net /Artix7/TDI: track 0.00 -> 88.9 mm, vias 0 -> 2
- net /Artix7/TDO: track 0.00 -> 82.1 mm, vias 0 -> 3
- net /Artix7/TCK: track 0.00 -> 78.8 mm, vias 0 -> 3
- net /Artix7/TMS: track 0.00 -> 78.4 mm, vias 0 -> 2
- net UART_MASTER_1_RX: track 0.00 -> 55.0 mm, vias 0 -> 2
- net /PowerSupply/PGOOD1V8: track 0.00 -> 54.5 mm, vias 0 -> 2
- net GP_BTN_1: track 0.00 -> 50.7 mm, vias 0 -> 2
- net UART_SLAVE_1_RX: track 0.00 -> 47.4 mm, vias 0 -> 2
- net I2C_MASTER_4_SCL: track 0.00 -> 47.2 mm, vias 0 -> 2
- net UART_SLAVE_2_RX: track 0.00 -> 47.0 mm, vias 0 -> 2
- net UART_MASTER_1_TX: track 0.00 -> 46.4 mm, vias 0 -> 2
- net SPI_SLAVE_4_MOSI: track 0.00 -> 45.9 mm, vias 0 -> 2
- net UART_SLAVE_2_TX: track 0.00 -> 44.8 mm, vias 0 -> 2
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- added copper zone on L4_Ground, net /Artix7/GNDADC
- added copper zone on B.Cu, net /Artix7/VCC1V0
- added copper zone on F.Cu, net /Artix7/VCC1V0
- added copper zone on B.Cu, net /Artix7/VCC1V8
- added copper zone on F.Cu, net /Artix7/VCC1V8
- added copper zone on B.Cu, net /Artix7/VCC3V3
- added copper zone on F.Cu, net /Artix7/VCC3V3
- added copper zone on F.Cu, net /PowerSupply/PWR_IN
Other:
- board size 100 x 120 mm -> 100 x 100 mm
- net class Default: via_dia 0.6096 -> 0.508
- rule pad_to_mask_clearance: 0.2 -> 0.2032
- rule via_min_size: 0.6096 -> 0.508

Commit message: layout finalizing
drc complete
Parts:
- added REF**: VIA - 2mil, InterNoC:VIA_2mil, F.Cu at (149.6, 131.4)
- added REF**: VIA - 2mil, InterNoC:VIA_2mil, F.Cu at (148.8, 129.8)
- added REF**: VIA - 2mil, InterNoC:VIA_2mil, F.Cu at (148.0, 129.8)
- added REF**: VIA - 2mil, InterNoC:VIA_2mil, F.Cu at (147.2, 129.8)
- added REF**: VIA - 2mil, InterNoC:VIA_2mil, F.Cu at (146.4, 129.8)
- added REF**: VIA - 2mil, InterNoC:VIA_2mil, F.Cu at (146.4, 130.6)
- added REF**: VIA - 2mil, InterNoC:VIA_2mil, F.Cu at (146.4, 131.4)
- added REF**: VIA - 2mil, InterNoC:VIA_2mil, F.Cu at (148.0, 133.0)
- added REF**: VIA - 2mil, InterNoC:VIA_2mil, F.Cu at (146.4, 133.0)
- added REF**: VIA - 2mil, InterNoC:VIA_2mil, F.Cu at (148.0, 132.2)
- added REF**: VIA - 2mil, InterNoC:VIA_2mil, F.Cu at (147.2, 132.2)
- added REF**: VIA - 2mil, InterNoC:VIA_2mil, F.Cu at (147.2, 130.6)
- added REF**: VIA - 2mil, InterNoC:VIA_2mil, F.Cu at (146.4, 132.2)
- added REF**: VIA - 2mil, InterNoC:VIA_2mil, F.Cu at (147.2, 133.0)
- added REF**: VIA - 2mil, InterNoC:VIA_2mil, F.Cu at (149.6, 133.0)
- added REF**: VIA - 2mil, InterNoC:VIA_2mil, F.Cu at (149.6, 132.2)
- added REF**: VIA - 2mil, InterNoC:VIA_2mil, F.Cu at (148.8, 132.2)
- added REF**: VIA - 2mil, InterNoC:VIA_2mil, F.Cu at (148.8, 133.0)
- added REF**: VIA - 2mil, InterNoC:VIA_2mil, F.Cu at (121.6, 133.0)
- added REF**: VIA - 2mil, InterNoC:VIA_2mil, F.Cu at (120.8, 133.0)
- added REF**: VIA - 2mil, InterNoC:VIA_2mil, F.Cu at (120.0, 133.0)
- added REF**: VIA - 2mil, InterNoC:VIA_2mil, F.Cu at (119.2, 133.0)
- added REF**: VIA - 2mil, InterNoC:VIA_2mil, F.Cu at (149.6, 130.6)
- added REF**: VIA - 2mil, InterNoC:VIA_2mil, F.Cu at (118.4, 133.0)
- added REF**: VIA - 2mil, InterNoC:VIA_2mil, F.Cu at (121.6, 132.2)
- added REF**: VIA - 2mil, InterNoC:VIA_2mil, F.Cu at (120.8, 132.2)
- added REF**: VIA - 2mil, InterNoC:VIA_2mil, F.Cu at (120.0, 132.2)
- added REF**: VIA - 2mil, InterNoC:VIA_2mil, F.Cu at (119.2, 132.2)
- added REF**: VIA - 2mil, InterNoC:VIA_2mil, F.Cu at (118.4, 132.2)
- added REF**: VIA - 2mil, InterNoC:VIA_2mil, F.Cu at (121.6, 131.4)
- added REF**: VIA - 2mil, InterNoC:VIA_2mil, F.Cu at (120.8, 131.4)
- added REF**: VIA - 2mil, InterNoC:VIA_2mil, F.Cu at (120.0, 131.4)
- added REF**: VIA - 2mil, InterNoC:VIA_2mil, F.Cu at (119.2, 131.4)
- added REF**: VIA - 2mil, InterNoC:VIA_2mil, F.Cu at (147.2, 131.4)
- added REF**: VIA - 2mil, InterNoC:VIA_2mil, F.Cu at (118.4, 131.4)
- added REF**: VIA - 2mil, InterNoC:VIA_2mil, F.Cu at (121.6, 130.6)
- added REF**: VIA - 2mil, InterNoC:VIA_2mil, F.Cu at (120.8, 130.6)
- added REF**: VIA - 2mil, InterNoC:VIA_2mil, F.Cu at (120.0, 130.6)
- added REF**: VIA - 2mil, InterNoC:VIA_2mil, F.Cu at (119.2, 130.6)
- added REF**: VIA - 2mil, InterNoC:VIA_2mil, F.Cu at (118.4, 130.6)
- added REF**: VIA - 2mil, InterNoC:VIA_2mil, F.Cu at (121.6, 129.8)
- added REF**: VIA - 2mil, InterNoC:VIA_2mil, F.Cu at (120.8, 129.8)
- added REF**: VIA - 2mil, InterNoC:VIA_2mil, F.Cu at (120.0, 129.8)
- added REF**: VIA - 2mil, InterNoC:VIA_2mil, F.Cu at (119.2, 129.8)
- added REF**: VIA - 2mil, InterNoC:VIA_2mil, F.Cu at (148.8, 131.4)
- added REF**: VIA - 2mil, InterNoC:VIA_2mil, F.Cu at (118.4, 129.8)
- added REF**: VIA - 2mil, InterNoC:VIA_2mil, F.Cu at (148.0, 131.4)
- added REF**: VIA - 2mil, InterNoC:VIA_2mil, F.Cu at (148.8, 130.6)
- added REF**: VIA - 2mil, InterNoC:VIA_2mil, F.Cu at (148.0, 130.6)
- added REF**: VIA - 2mil, InterNoC:VIA_2mil, F.Cu at (149.6, 129.8)
- moved C6 2.24 mm to (85.6, 132.6), turned to 0 degrees
- moved C1 1.70 mm to (85.0, 130.0), turned to 0 degrees
Routing:
- net GND: track 320.5 -> 325.8 mm, vias 234 -> 236
- net UART_MASTER_1_RX: track 55.0 -> 51.6 mm
- net /PowerSupply/PGOOD1V8: track 54.5 -> 57.2 mm
- net Net-(J31-Pad3): track 13.6 -> 11.1 mm
- net Net-(J31-Pad5): track 13.6 -> 11.3 mm
- net Net-(C6-Pad1): track 2.45 -> 4.35 mm
- net /PowerSupply/PGOOD1V0: track 39.1 -> 40.7 mm
- net /Artix7/GNDADC: track 9.53 -> 11.0 mm
- net /PowerSupply/PGOOD: track 25.6 -> 24.2 mm
- net Net-(R7-Pad2): track 12.1 -> 10.7 mm
- net Net-(J31-Pad6): track 10.2 -> 8.98 mm
- net I2C_MASTER_1_SCL: track 41.2 -> 40.0 mm
- net /Artix7/VCC3V3: track 43.0 -> 44.0 mm
- net /Artix7/VCC1V8: track 3.54 -> 4.53 mm
- net I2C_MASTER_2_SCL: track 41.5 -> 40.6 mm
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- added copper zone on F.Cu, net GND

Commit message: fin
Parts:
- added G***: LOGO, InterNoC:lclogic_logo_9.5x1.9, F.Cu at (90.3, 102.3)
- added G***: LOGO, InterNoC:InterNoC_logo, F.Cu at (91.5, 96.4)
- added REF**: VIA - 2mil, InterNoC:VIA_2mil, F.Cu at (80.1, 129.6)
- added REF**: VIA - 2mil, InterNoC:VIA_2mil, F.Cu at (79.3, 129.6)
- added REF**: VIA - 2mil, InterNoC:VIA_2mil, F.Cu at (80.1, 128.8)
- added REF**: VIA - 2mil, InterNoC:VIA_2mil, F.Cu at (79.3, 128.8)
- added REF***: OSHW-Logo2_7.3x6mm_SilkScreen, Symbols:OSHW-Logo2_7.3x6mm_SilkScreen, F.Cu at (146.0, 115.9)
- I2C MASTER 1: renamed from J8
- I2C MASTER 2: renamed from J9
- I2C MASTER 3: renamed from J10
- I2C MASTER 4: renamed from J11
- I2C SLAVE 1: renamed from J16
- I2C SLAVE 2: renamed from J17
- I2C SLAVE 3: renamed from J18
- I2C SLAVE 4: renamed from J19
- I2C SLAVE 5: renamed from J24
- I2C SLAVE 6: renamed from J25
- I2C SLAVE 7: renamed from J26
- I2C SLAVE 8: renamed from J27
- SPI MASTER 1: renamed from J13
- SPI MASTER 2: renamed from J14
- SPI MASTER 3: renamed from J15
- SPI SLAVE 1: renamed from J21
- SPI SLAVE 2 : renamed from J22
- SPI SLAVE 3: renamed from J23
- SPI SLAVE 4: renamed from J29
- SPI SLAVE 5: renamed from J30
- SPI SLAVE 6: renamed from J31
- UART MASTER : renamed from J12
- UART SLAVE 1: renamed from J20
- UART SLAVE 2: renamed from J28
- moved C35 1.45 mm to (98.0, 91.5)
- moved C104 1.40 mm to (125.6, 80.7)
- moved C106 1.40 mm to (124.2, 80.7)
- moved C56 1.35 mm to (98.0, 90.1)
- moved C43 0.11 mm to (93.3, 87.7)
- moved L4 0.05 mm to (127.3, 81.3)
- renumbered J6 to TP1V0, J5 to TP1V8, J7 to TP3V3
Other:
- board text added: "+"
- board text added: "-"
- board text added: "1-SDA"
- board text added: "1-TX"
- board text added: "2-GND"
- board text added: "2-RX"
- board text added: "2-SCL"
- board text added: "3-GND"
- board text added: "4-MOSI"
- board text added: "5V IN ONLY"
- board text added: "6-MISO"
- board text added: "ADDRESSES:"
- board text added: "CS-5"
- board text added: "Conf Done"
- board text added: "Designed by Chris Gkiokas"
- board text added: "I2C:"
- board text added: "JTAG"
- board text added: "MASTERS:"
- board text added: "NC-1"
- board text added: "OFF/ON"
- board text added: "PINOUTS:"
- board text added: "Power ON"
- board text added: "REV A"
- board text added: "Reset Config"
- board text added: "S/N:"
- board text added: "SCLK-3"
- board text added: "SLAVES:"
- board text added: "SPI 1:0x00 SPI 2:0x01 SPI 3:0x02 SPI 4:0x03 SPI 5:0x04 SPI 6:0x05 I2C 1:0x06 I2C 2:0x07 I2C 3:0x08 I2C 4:0x09 I2C 5:0x0A I2C 6:0x0B I2C 7:0x0C I2C 8:0x0D UART 1:0x0E UART 2:0x0F"
- board text added: "SPI 1:0x10 SPI 2:0x11 SPI 3:0x12 I2C 1:0x13 I2C 2:0x14 I2C 3:0x15 I2C 4:0x16 UART:0x17"
- board text added: "SPI:"
- board text added: "UART:"
- board text added: "center (+)"
